File: pcb/battery_controller.sch (KiCad schematic (older format))
At the start: 65 parts

Commit message: adding battery controller
Parts:
- removed C? (x2): 0.047uF, Capacitor_SMD:C_0603_1608Metric, symbol Device:C
- removed C?: 33pF, Capacitor_SMD:C_0603_1608Metric, symbol Device:C
- removed C?: 1000pF, Capacitor_SMD:C_0603_1608Metric, symbol Device:C
- removed C? (x2): 0.01uF, Capacitor_SMD:C_0603_1608Metric, symbol Device:C
- removed C? (x2): 0.033uF, Capacitor_SMD:C_0603_1608Metric, symbol Device:C
- removed C? (x2): 1uF, Capacitor_SMD:C_0603_1608Metric, symbol Device:C
- removed C?: 2.2uF, Capacitor_SMD:C_0603_1608Metric, symbol Device:C
- removed C?: 1800pF, Capacitor_SMD:C_0603_1608Metric, symbol Device:C
- removed C?: 15pF, Capacitor_SMD:C_0603_1608Metric, symbol Device:C
- removed C?: 680pF, Capacitor_SMD:C_0603_1608Metric, symbol Device:C
- removed C? (x2): 150pF, Capacitor_SMD:C_0603_1608Metric, symbol Device:C
- removed C?: 10uF, Capacitor_SMD:C_0603_1608Metric, symbol Device:C
- removed C?: 0.1uF, Capacitor_SMD:C_0603_1608Metric, symbol Device:C
- removed C? (x3): 100pF, Capacitor_SMD:C_0603_1608Metric, symbol Device:C
- removed C? (x13): 10uF, Capacitor_SMD:C_0805_2012Metric, symbol Device:C
- removed C? (x2): 33uF, Capacitor_SMD:C_0805_2012Metric, symbol Device:CP
- removed D?: D_Schottky, symbol Device:D_Schottky
- removed D?: D_Zener, symbol Device:D_Zener
- removed J?: MegaFit 2x1, RespiraWorks_Std:Molex_Mega-Fit_76829-0102_2x01_P5.70mm_Vertical, symbol Connector:Conn_01x02_Male
- removed J?: MegaFit 2x2, RespiraWorks_Std:Molex_Mega-Fit_76829-0104_2x02_P5.70mm_Vertical, symbol Connector:Conn_01x04_Male
- removed L?: SRP1038A-3R3M, symbol RespiraWorks_Std:SRP1038A-3R3M
- removed Q?: CSD25402Q3A, Package_SON:VSON-8_3.3x3.3mm_P0.65mm_NexFET, symbol RespiraWorks_Std:CSD25402Q3A
- removed Q? (x4): CSD17304Q3, Package_SON:VSON-8_3.3x3.3mm_P0.65mm_NexFET, symbol RespiraWorks_Std:CSD17304Q3
- removed R? (x2): 0.01, Capacitor_SMD:C_1206_3216Metric, symbol Device:R
- removed R? (x3): 4.99, Resistor_SMD:R_0603_1608Metric, symbol Device:R
- removed R? (x3): 10k, Resistor_SMD:R_0603_1608Metric, symbol Device:R
- removed R?: 40.2k, Resistor_SMD:R_0603_1608Metric, symbol Device:R
- removed R? (x2): 10, Resistor_SMD:R_0603_1608Metric, symbol Device:R
- removed R?: 78.7k, Resistor_SMD:R_0603_1608Metric, symbol Device:R
- removed R? (x2): 100k, Resistor_SMD:R_0603_1608Metric, symbol Device:R
- removed R?: 0, Resistor_SMD:R_0603_1608Metric, symbol Device:R
- removed R?: 68k, Resistor_SMD:R_0603_1608Metric, symbol Device:R
- removed R? (x2): 169k, Resistor_SMD:R_0603_1608Metric, symbol Device:R
Connections:
- net labels removed: BAT_N, BAT_P, CHG_OK, EN_OTG, GND, IADPT, IBAT, ILIM_HIZ, PSYS, REGN, VDDA, VIN_12V, VLOGIC, VSYS
- wire segments 162 -> 2
- no-connect marks 2 -> 0
Other:
- note added: "Design notes:\n- 8.2A max current, 19V input\n- Inductor selection: Isat 9.1A, 3.3uH\n- Wurth 7443330330 or Bourns SRP1038A-3R3M\n- Voltage will range from 10.8V to 12.6V for 3s Li-Ion battery\n- 11.5 to 13.0V for SLA (lead acid)\n- \n"
- note removed: "55% of VDDA to set 3s battery"
- note removed: "Design notes:\n- 8.2A max current, 19V input\n- Inductor selection: Isat 9.1A, 3.3uH\n- Wurth 7443330330 or Bourns SRP1038A-3R3M (OPL alt: MWSA1004-3R3MT)\n- Voltage will range from 10.8V to 12.6V for 3s Li-Ion battery\n- 11.5 to 13.0V for SLA (lead acid)\n- N-CH FET: CSD17304Q3 (OPL) or BSZ050N03LSGATMA1 (OPL)\n- P-CH FET: CSD25402Q3A (OPL) or CSD25404Q3T (OPL)\n"
- note removed: "IADPT pulldown resistance\nfor inductance detection:\n1uH 93k\n2.2uH 137k\n3.3uH 169k"
- note removed: "Pin count to prevent incorrect mating"
- note removed: "TODO: add NO BAT detection"
- note removed: "TODO: input protection"
- note removed: "VDDA = 6.0V"
- note removed: "V_ilim = 3.57V > ILIM = 6400mA\nShort ILIM_HIZ to GND to shut off all power"
