File: pcb/battery_controller.sch (KiCad schematic (older format))
At the start: 6 parts

Commit message: adding battery controller
Parts:
- removed C?: 10uF, Capacitor_SMD:C_0603_1608Metric, symbol Device:C
- removed D?: 20V, Diode_SMD:D_SMC, symbol Device:D_Zener
- removed F? (x2): Fuse 10A, symbol Device:Fuse
- removed J?: MegaFit 2x2, RespiraWorks_Std:Molex_Mega-Fit_76829-0104_2x02_P5.70mm_Vertical, symbol Connector:Conn_01x04_Male
- removed J?: MegaFit 2x1, RespiraWorks_Std:Molex_Mega-Fit_76829-0102_2x01_P5.70mm_Vertical, symbol Connector:Conn_01x02_Male
- added U?: BQ25713, Package_DFN_QFN:Texas_S-PWQFN-N32_EP2.8x2.8mm_ThermalVias, symbol RespiraWorks:BQ25713
Connections:
- net labels removed: 12VOUT, BAT_ALRT, BAT_N, BAT_P, GND, PG_12V, PMON_ACOK, PMON_IADP, PMON_IBAT, PMON_PSYS, POWER_SW_N, POWER_SW_P, VIN_ADP, VLOGIC
- wire segments 32 -> 2
Other:
- note added: "Design notes:\n- 8.2A max current, 19V input\n- Inductor selection: Isat 9.1A, 3.3uH\n- Wurth 7443330330 or Bourns SRP1038A-3R3M\n- Voltage will range from 10.8V to 12.6V for 3s Li-Ion battery\n- 11.5 to 13.0V for SLA (lead acid)\n- \n"
