File: pcb/battery_balancer.sch (KiCad schematic (older format))
At the start: 27 parts

Commit message: restructured schematic to place charger, balancer, and VSYS supply on separate sheets
Parts:
- removed C? (x5): 0.01uF, Capacitor_SMD:C_0603_1608Metric, symbol Device:C
- removed C? (x2): 0.1uF, Capacitor_SMD:C_0603_1608Metric, symbol Device:C
- removed C? (x4): 0.47uF, Capacitor_SMD:C_0603_1608Metric, symbol Device:C
- removed J?: Conn_01x05_Male, symbol Connector:Conn_01x05_Male
- removed Q? (x2): CSD17304Q3, Package_SON:VSON-8_3.3x3.3mm_P0.65mm_NexFET, symbol RespiraWorks_Std:CSD17304Q3
- removed R?: 0.005, Resistor_SMD:R_1206_3216Metric, symbol Device:R
- removed R? (x4): 49.9, Resistor_SMD:R_1206_3216Metric, symbol Device:R
- removed R?: 10, RespiraWorks_Std:R_0603_1608Metric, symbol Device:R
- removed R? (x2): 1k, RespiraWorks_Std:R_0603_1608Metric, symbol Device:R
- removed R?: 2k, RespiraWorks_Std:R_1206_3216Metric, symbol Device:R
- removed R? (x2): 100, RespiraWorks_Std:R_0603_1608Metric, symbol Device:R
- removed TH?: 10k, Resistor_SMD:R_0603_1608Metric, symbol Device:Thermistor_NTC
- removed U?: MAX17320G20+, Package_DFN_QFN:WQFN-24-1EP_4x4mm_P0.5mm_EP2.6x2.6mm, symbol RespiraWorks:MAX17320G20+
Connections:
- net labels removed: ALRT, BAT_N, BAT_P, GND, SCL, SDA, SYS_N, SYS_P
- wire segments 72 -> 0
- no-connect marks 3 -> 0
Other:
- note removed: "Balancing current: 100mA MAX"
- note removed: "Battery Balancing Connector"
