File: pcb/battery_charger.sch (KiCad schematic (older format))
At the start: 56 parts

Commit message: restructured schematic to place charger, balancer, and VSYS supply on separate sheets
Parts:
- removed C?: 100pF, Capacitor_SMD:C_0603_1608Metric, symbol Device:C
- removed C?: 0.01uF, Capacitor_SMD:C_0603_1608Metric, symbol Device:C
- removed D?: BAT54C, Package_TO_SOT_SMD:SOT-23, symbol Diode:BAT54C
- removed R?: 10k, Resistor_SMD:R_0603_1608Metric, symbol Device:R
- removed R? (x2): 316k, Resistor_SMD:R_0603_1608Metric, symbol Device:R
- removed R? (x2): 100k, Resistor_SMD:R_0603_1608Metric, symbol Device:R
- removed R?: 0, Resistor_SMD:R_0603_1608Metric, symbol Device:R
- removed R?: 3M, Resistor_SMD:R_0603_1608Metric, symbol Device:R
- added D? (x2): D_Schottky, symbol Device:D_Schottky
- added R?: 169k, Resistor_SMD:R_0603_1608Metric, symbol Device:R
- C?: value 0.01uF -> 100pF
- R? (x2): footprint RespiraWorks_Std:R_1206_3216Metric -> Capacitor_SMD:C_1206_3216Metric
- R?: value 30.1k -> 169k
Connections:
- net labels added: BAT_P
- net labels removed: PACK_P
- wire segments 146 -> 133
Other:
- note added: "Design notes:\n- 6.3A max current, 19V input\n- Inductor selection: Isat 9.1A, 3.3uH\n- Wurth 7443330330 or Bourns SRP1038A-3R3M (OPL alt: MWSA1004-3R3MT)\n- Voltage will range from 10.8V to 12.6V for 3s Li-Ion battery\n- 11.5 to 13.0V for SLA (lead acid)\n- N-CH FET: CSD17304Q3 (OPL) or BSZ050N03LSGATMA1 (OPL)\n- P-CH FET: CSD25402Q3A (OPL) or CSD25404Q3T (OPL)\n"
- note added: "V_ilim = 3.57V > ILIM = 6400mA\nShort ILIM_HIZ to GND to shut off all power"
- note removed: "Design notes:\n- 6.3A max current, 20V input\n- Inductor selection: Isat 9.1A, 3.3uH\n- Wurth 7443330330 or Bourns SRP1038A-3R3M (OPL alt: MWSA1004-3R3MT)\n- Voltage will range from 12V to 16.8V for 4s Li-Ion battery\n- 11.5 to 13.0V for SLA (lead acid)\n- N-CH FET: CSD17304Q3 (OPL) or BSZ050N03LSGATMA1 (OPL)\n- P-CH FET: CSD25402Q3A (OPL) or CSD25404Q3T (OPL)\n"
- note removed: "Optional: R between CMPIN and\nCMPOUT sets hysteresis\n(not req'd when comparator \npolarity set to LOW)"
- note removed: "PMON default is 1uA/W\nIBAT and IADT are voltage outputs\n"
- note removed: "Threshold here is 2.3V, max of 7V\nnBATPRES asserted when BAT_P over 9.6V\nReused ILIM resistor values to reduce BOM."
- note removed: "V_ilim = 20*IPDM*Rac\nV_ilim = 1.29V -> 6.45A"
- moved on the sheet: C?
